Commit message: Refactor controller parameters and update URDF for improved simulation performance

File: urdf/amr.urdf.xacro (robot description, xacro)
@@ -23,9 +23,9 @@
   <link name="base_link">
     <inertial>
-      <origin xyz="-0.0513 0 0.104" rpy="0 0 0"/>
-      <mass value="5.8"/>
-      <inertia ixx="0.0770" ixy="0.0" ixz="0.0"
-               iyy="0.1624" iyz="0.0"
-               izz="0.2177"/>
+      <origin xyz="0 0 0" rpy="0 0 0"/>
+      <mass value="18.71"/>
+      <inertia ixx="0.3986" ixy="0"      ixz="0"
+               iyy="1.092"  iyz="0"
+               izz="1.337"/>
     </inertial>
     <visual>
@@ -57,26 +57,27 @@
     Collision: kept as cylinder (more stable than mesh for physics).
   -->
-  <link name="front_left_wheel">
-    <inertial>
-      <mass value="0.108"/>
-      <origin xyz="0 0 0"/>
-      <inertia ixx="0.000174" ixy="0" ixz="0"
-               iyy="0.000174" iyz="0"
-               izz="0.000278"/>
-    </inertial>
-    <visual>
-      <origin xyz="0 0 0" rpy="0 0 0"/>
-      <geometry>
-        <mesh filename="package://amr_description/meshes/Front_Left_Wheel.STL"/>
-      </geometry>
-      <material name="light_gray"/>
-    </visual>
-    <collision>
-      <origin xyz="0 0 0" rpy="0 0 0"/>
-      <geometry>
-        <cylinder radius="0.065" length="0.05"/>
-      </geometry>
-    </collision>
-  </link>
+    <link name="front_left_wheel">
+        <inertial>
+            <origin xyz="0.0 0.0 0.0" rpy="0.0 0.0 0.0"/>
+            <mass value="1.0"/>
+            <inertia ixx="0.1" ixy="0.0" ixz="0.0" iyy="0.1" iyz="0.0" izz="0.1"/>
+        </inertial>
+        <visual name="">
+            <origin xyz="0.0 0.0 0.0" rpy="0.0 0.0 0.0"/>
+            <geometry>
+                <mesh filename="package://amr_description/meshes/Front_Left_Wheel.STL"/>
+            </geometry>
+            <material name="">
+                <color rgba="0.5 0.2 0.1 1.0"/>
+                <texture filename=""/>
+            </material>
+        </visual>
+        <collision>
+            <origin xyz="0.0 0.0 0.0" rpy="0.0 0.0 0.0"/>
+            <geometry>
+                <cylinder radius="0.065" length="0.05"/>
+            </geometry>
+        </collision>
+    </link>
   <joint name="front_left_wheel_joint" type="continuous">
     <parent link="base_link"/>
@@ -87,19 +88,17 @@
   </joint>
   <gazebo reference="front_left_wheel">
-    <material>Gazebo/Grey</material>
     <collision>
       <surface>
         <friction>
           <ode>
-            <mu>10.0</mu>
-            <mu2>10.0</mu2>
-            <slip1>0.0</slip1>
-            <slip2>0.0</slip2>
+            <mu>1.0</mu>
+            <mu2>0.01</mu2>
+            <fdir1>1 0 0</fdir1>
           </ode>
         </friction>
         <contact>
           <ode>
-            <kp>1e7</kp>
-            <kd>100.0</kd>
+            <kp>1e6</kp>
+            <kd>10.0</kd>
           </ode>
         </contact>
@@ -117,26 +116,27 @@
     for differential drive. No axis swap or multiplier hack needed.
   -->
-  <link name="front_right_wheel">
-    <inertial>
-      <mass value="0.108"/>
-      <origin xyz="0 0 0"/>
-      <inertia ixx="0.000174" ixy="0" ixz="0"
-               iyy="0.000174" iyz="0"
-               izz="0.000278"/>
-    </inertial>
-    <visual>
-      <origin xyz="0 0 0" rpy="0 0 0"/>
-      <geometry>
-        <mesh filename="package://amr_description/meshes/Front_Right_Wheel.STL"/>
-      </geometry>
-      <material name="light_gray"/>
-    </visual>
-    <collision>
-      <origin xyz="0 0 0" rpy="0 0 0"/>
-      <geometry>
-        <cylinder radius="0.065" length="0.05"/>
-      </geometry>
-    </collision>
-  </link>
+    <link name="front_right_wheel">
+        <inertial>
+            <origin xyz="0.0 0.0 0.0" rpy="0.0 0.0 0.0"/>
+            <mass value="1.0"/>
+            <inertia ixx="0.1" ixy="0.0" ixz="0.0" iyy="0.1" iyz="0.0" izz="0.1"/>
+        </inertial>
+        <visual name="">
+            <origin xyz="0.0 0.0 0.0" rpy="0.0 0.0 0.0"/>
+            <geometry>
+                <mesh filename="package://amr_description/meshes/Front_Right_Wheel.STL"/>
+            </geometry>
+            <material name="">
+                <color rgba="0.5 0.2 0.1 1.0"/>
+                <texture filename=""/>
+            </material>
+        </visual>
+        <collision>
+            <origin xyz="0.0 0.0 0.0" rpy="0.0 0.0 0.0"/>
+            <geometry>
+                <cylinder radius="0.065" length="0.05"/>
+            </geometry>
+        </collision>
+    </link>
   <joint name="front_right_wheel_joint" type="continuous">
     <parent link="base_link"/>
@@ -147,19 +147,17 @@
   </joint>
   <gazebo reference="front_right_wheel">
-    <material>Gazebo/Grey</material>
     <collision>
       <surface>
         <friction>
           <ode>
-            <mu>10.0</mu>
-            <mu2>10.0</mu2>
-            <slip1>0.0</slip1>
-            <slip2>0.0</slip2>
+            <mu>1.0</mu>
+            <mu2>0.01</mu2>
+            <fdir1>1 0 0</fdir1>
           </ode>
         </friction>
         <contact>
           <ode>
-            <kp>1e7</kp>
-            <kd>100.0</kd>
+            <kp>1e6</kp>
+            <kd>10.0</kd>
           </ode>
         </contact>
@@ -170,26 +168,27 @@
   <!-- BACK LEFT WHEEL                                              -->
   <!-- =========================================================== -->
-  <link name="back_left_wheel">
-    <inertial>
-      <mass value="0.108"/>
-      <origin xyz="0 0 0"/>
-      <inertia ixx="0.000174" ixy="0" ixz="0"
-               iyy="0.000174" iyz="0"
-               izz="0.000278"/>
-    </inertial>
-    <visual>
-      <origin xyz="0 0 0" rpy="0 0 0"/>
-      <geometry>
-        <mesh filename="package://amr_description/meshes/Back_Left_Wheel.STL"/>
-      </geometry>
-      <material name="light_gray"/>
-    </visual>
-    <collision>
-      <origin xyz="0 0 0" rpy="0 0 0"/>
-      <geometry>
-        <cylinder radius="0.065" length="0.05"/>
-      </geometry>
-    </collision>
-  </link>
+    <link name="back_left_wheel">
+        <inertial>
+            <origin xyz="0.0 0.0 0.0" rpy="0.0 0.0 0.0"/>
+            <mass value="1.0"/>
+            <inertia ixx="0.1" ixy="0.0" ixz="0.0" iyy="0.1" iyz="0.0" izz="0.1"/>
+        </inertial>
+        <visual name="">
+            <origin xyz="0.0 0.0 0.0" rpy="0.0 0.0 0.0"/>
+            <geometry>
+              <mesh filename="package://amr_description/meshes/Back_Left_Wheel.STL"/>
+            </geometry>
+            <material name="">
+                <color rgba="0.5 0.2 0.1 1.0"/>
+                <texture filename=""/>
+            </material>
+        </visual>
+        <collision>
+            <origin xyz="0.0 0.0 0.0" rpy="0.0 0.0 0.0"/>
+            <geometry>
+                <cylinder radius="0.065" length="0.05"/>
+            </geometry>
+        </collision>
+    </link>
   <joint name="back_left_wheel_joint" type="continuous">
     <parent link="base_link"/>
@@ -200,19 +199,17 @@
   </joint>
   <gazebo reference="back_left_wheel">
-    <material>Gazebo/Grey</material>
     <collision>
       <surface>
         <friction>
           <ode>
-            <mu>10.0</mu>
-            <mu2>10.0</mu2>
-            <slip1>0.0</slip1>
-            <slip2>0.0</slip2>
+            <mu>1.0</mu>
+            <mu2>0.01</mu2>
+            <fdir1>1 0 0</fdir1>
           </ode>
         </friction>
         <contact>
           <ode>
-            <kp>1e7</kp>
-            <kd>100.0</kd>
+            <kp>1e6</kp>
+            <kd>10.0</kd>
           </ode>
         </contact>
@@ -229,26 +226,27 @@
     mirrored rpy as front right to keep both right wheels consistent.
   -->
-  <link name="back_right_wheel">
-    <inertial>
-      <mass value="0.108"/>
-      <origin xyz="0 0 0"/>
-      <inertia ixx="0.000174" ixy="0" ixz="0"
-               iyy="0.000174" iyz="0"
-               izz="0.000278"/>
-    </inertial>
-    <visual>
-      <origin xyz="0 0 0" rpy="0 0 0"/>
-      <geometry>
-        <mesh filename="package://amr_description/meshes/Back_Right_Wheel.STL"/>
-      </geometry>
-      <material name="light_gray"/>
-    </visual>
-    <collision>
-      <origin xyz="0 0 0" rpy="0 0 0"/>
-      <geometry>
-        <cylinder radius="0.065" length="0.05"/>
-      </geometry>
-    </collision>
-  </link>
+    <link name="back_right_wheel">
+        <inertial>
+            <origin xyz="0.0 0.0 0.0" rpy="0.0 0.0 0.0"/>
+            <mass value="1.0"/>
+            <inertia ixx="0.1" ixy="0.0" ixz="0.0" iyy="0.1" iyz="0.0" izz="0.1"/>
+        </inertial>
+        <visual name="">
+            <origin xyz="0.0 0.0 0.0" rpy="0.0 0.0 0.0"/>
+            <geometry>
+                <mesh filename="package://amr_description/meshes/Back_Right_Wheel.STL"/>
+            </geometry>
+            <material name="">
+                <color rgba="0.5 0.2 0.1 1.0"/>
+                <texture filename=""/>
+            </material>
+        </visual>
+        <collision>
+            <origin xyz="0.0 0.0 0.0" rpy="0.0 0.0 0.0"/>
+            <geometry>
+                <cylinder radius="0.065" length="0.05"/>
+            </geometry>
+        </collision>
+    </link>
   <joint name="back_right_wheel_joint" type="continuous">
     <parent link="base_link"/>
@@ -259,19 +257,17 @@
   </joint>
   <gazebo reference="back_right_wheel">
-    <material>Gazebo/Grey</material>
     <collision>
       <surface>
         <friction>
           <ode>
-            <mu>10.0</mu>
-            <mu2>10.0</mu2>
-            <slip1>0.0</slip1>
-            <slip2>0.0</slip2>
+            <mu>1.0</mu>
+            <mu2>0.01</mu2>
+            <fdir1>1 0 0</fdir1>
           </ode>
         </friction>
         <contact>
           <ode>
-            <kp>1e7</kp>
-            <kd>100.0</kd>
+            <kp>1e6</kp>
+            <kd>10.0</kd>
           </ode>
         </contact>
